File: hardware/stm32-head/stepper_drivers.kicad_sch (KiCad schematic)
At the start: 64 parts, among them J10 STEPPER4, J17 STEPPER6, J18 STEPPER5, J7 STEPPER1, J8 STEPPER2, J9 STEPPER3, U10 STSPIN220, U11 STSPIN220, U12 STSPIN220, U9 STSPIN220

Commit message: Board fixes
Parts:
- added C23, C24: 10uF, Capacitor_SMD:CP_Elec_6.3x5.9, symbol Device:C_Polarized
- C15, C17, C19, C21: footprint Capacitor_Tantalum_SMD:CP_EIA-2012-12_Kemet-R -> Capacitor_Tantalum_SMD:CP_EIA-3216-10_Kemet-I
Connections:
- net +12V: now also C23.1, C24.1
- net GND: now also C23.2, C24.2
- net at U9.10 (OUTB1): now also J7.3 (Pin_3); no longer J7.2 (Pin_2)
- net at U9.3 (OUTA1): now also J7.1 (Pin_1); no longer J7.4 (Pin_4)
- net at U9.5 (OUTA2): now also J7.2 (Pin_2); no longer J7.3 (Pin_3)
- net at U9.8 (OUTB2): now also J7.4 (Pin_4); no longer J7.1 (Pin_1)
- net at J9.1 (Pin_1): now also U11.3 (OUTA1); no longer U11.8 (OUTB2)
- net at J9.2 (Pin_2): now also U11.5 (OUTA2); no longer U11.10 (OUTB1)
- net at J9.3 (Pin_3): now also U11.10 (OUTB1); no longer U11.5 (OUTA2)
- net at J9.4 (Pin_4): now also U11.8 (OUTB2); no longer U11.3 (OUTA1)
- net at U12.10 (OUTB1): now also J10.3 (Pin_3); no longer J10.2 (Pin_2)
- net at U12.3 (OUTA1): now also J10.1 (Pin_1); no longer J10.4 (Pin_4)
- net at U12.5 (OUTA2): now also J10.2 (Pin_2); no longer J10.3 (Pin_3)
- net at U12.8 (OUTB2): now also J10.4 (Pin_4); no longer J10.1 (Pin_1)
- net at J8.1 (Pin_1): now also U10.3 (OUTA1); no longer U10.8 (OUTB2)
- net at J8.2 (Pin_2): now also U10.5 (OUTA2); no longer U10.10 (OUTB1)
- net at J8.3 (Pin_3): now also U10.10 (OUTB1); no longer U10.5 (OUTA2)
- net at J8.4 (Pin_4): now also U10.8 (OUTB2); no longer U10.3 (OUTA1)
Other:
- note added: "To DRV8825"

Commit message: HW fixes
Parts:
- added Q?: AO3400A, Package_TO_SOT_SMD:SOT-23, symbol Transistor_FET:AO3400A
- added R68, R69, R70, R71, R72: 20K, Resistor_SMD:R_0603_1608Metric, symbol Device:R
- added R?: 5K, Resistor_SMD:R_0603_1608Metric, symbol Device:R
- added R?: 100, Resistor_SMD:R_0603_1608Metric, symbol Device:R
Connections:
- net +3.3V: now also R31.2; no longer R31.1, R33.1, R35.1, R37.1
- net GND: now also R33.1, R35.1, R37.1, Q?.2 (S), R68.1, R69.1, R70.1, R71.1, R72.1, R?.1
- net STEP_ENA: now also R31.1, Q?.1 (G), R?.2; no longer A1.9 (~{EN}), A2.9 (~{EN}), R31.2, R33.2, R35.2, R37.2
- net at JP8.2 (B), U12.16 (MODE1): now also R71.2
- net at JP3.2 (B), U9.15 (MODE2): now also R68.2
- net at JP2.2 (B), U9.16 (MODE1): now also R72.2
- net at JP5.2 (B), U10.15 (MODE2): now also R33.2
- net at JP9.2 (B), U12.15 (MODE2): now also R37.2
- net at JP7.2 (B), U11.15 (MODE2): now also R35.2
- net at JP6.2 (B), U11.16 (MODE1): now also R70.2
- net at JP4.2 (B), U10.16 (MODE1): now also R69.2
- new net: Q?.3 (D), R?.2
- new net POLOLU_ENA: A1.9 (~{EN}), A2.9 (~{EN}), R?.1
Other:
- moved on the sheet: C10, C11, C12, C13, C14, C15, C16, C17, C18, C19, C20, C21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

Commit message: Some tweaks
Parts:
- removed Q?: AO3400A, Package_TO_SOT_SMD:SOT-23, symbol Transistor_FET:AO3400A
- removed R?: 5K, Resistor_SMD:R_0603_1608Metric, symbol Device:R
- added Q6: AO3401A, Package_TO_SOT_SMD:SOT-23, symbol Transistor_FET:AO3401A
- added R73: 100, Resistor_SMD:R_0603_1608Metric, symbol Device:R
- R31: value 20K -> 10K
- R74: renamed from R?; value 100 -> 47K
Connections:
- net +3.3V: now also R73.1
- net GND: now also R74.1
- net POLOLU_ENA: now also R74.2, Q6.3 (D); no longer R74.1
- net STEP_ENA: now also Q6.1 (G)
- new net: Q6.2 (S), R73.2
Other:
- moved on the sheet: A1, A2, C23, C24, J17, J18, R31, R74
