File: hardware/stm32-head/stm32-head.kicad_pcb (KiCad board)
At the start: 2 copper layers, 80 x 60 mm, 163 parts, among them J1 POWER, J10 STEPPER4, J11 SWD, J12 LIMIT_4, J13 SOLENOID1, J14 SOLENOID2, J15 SOLENOID3, J16 SOLENOID4, J17 STEPPER6, J18 STEPPER5, J19 LED, J2 RS-485, J3 LIMIT_1, J4 LIMIT_2, J5 LIMIT_3, J6 LIGHT, J7 STEPPER1, J8 STEPPER2, J9 STEPPER3, Q1 IRF540N, Q2 AO3400A, Q3 AO3400A, Q4 AO3400A, Q5 AO3400A, SW1 RESET, U1 LM2596S-ADJ, U10 STSPIN220, U11 STSPIN220, U12 STSPIN220, U13 PC817, U14 PC817, U15 PC817, U16 PC817, U17 PC817, U2 STM32F103C8Tx, U3 AMS1117-3.3, U4 MAX483E, U5 PC817, U6 PC817, U7 PC817, U8 PC817, U9 STSPIN220, Y1 8Mhz

Commit message: Board fixes
Parts:
- removed U13, U14, U15, U16, U17: PC817, Package_DIP:SMDIP-4_W9.53mm
- added C23: 10uF, Capacitor_SMD:CP_Elec_6.3x5.9, F.Cu at (123.6, 56.4)
- added C24: 10uF, Capacitor_SMD:CP_Elec_6.3x5.9, F.Cu at (123.7, 40.6)
- added FID1: Fiducial, Fiducial:Fiducial_0.5mm_Mask1mm, F.Cu at (59.9, 78.9)
- added FID2: Fiducial, Fiducial:Fiducial_0.5mm_Mask1mm, F.Cu at (63.6, 32.0)
- added FID3: Fiducial, Fiducial:Fiducial_0.5mm_Mask1mm, F.Cu at (131.1, 29.0)
- added FID4: Fiducial, Fiducial:Fiducial_0.5mm_Mask1mm, F.Cu at (120.9, 83.1)
- added R65: 1K, Resistor_SMD:R_0603_1608Metric, F.Cu at (74.8, 56.3)
- added R66: 10K, Resistor_SMD:R_0603_1608Metric, F.Cu at (74.8, 57.8)
- added R67: 32K, Resistor_SMD:R_0603_1608Metric, F.Cu at (77.9, 57.8)
- C15, C17, C19, C21: footprint Capacitor_Tantalum_SMD:CP_EIA-2012-12_Kemet-R -> Capacitor_Tantalum_SMD:CP_EIA-3216-10_Kemet-I
- Q1: footprint Package_TO_SOT_THT:TO-220-3_Vertical -> Package_TO_SOT_SMD:TO-252-3_TabPin2
- R2, R61, R62, R63, R64: value 100 -> 510
- R4, R5: value 100 -> 1K
- R49, R50, R51, R52, R9: value 100 -> 150
- U6: value PC817 -> TL431DBZ; footprint Package_DIP:SMDIP-4_W9.53mm -> Package_TO_SOT_SMD:SOT-23
- U7, U8: value PC817 -> TLP291-4; footprint Package_DIP:SMDIP-4_W9.53mm -> Package_SO:SOIC-16_4.55x10.3mm_P1.27mm
- Y1: footprint Crystal:Crystal_SMD_5032-2Pin_5.0x3.2mm -> Crystal:Crystal_SMD_3225-4Pin_3.2x2.5mm
- moved U8 39.6 mm to (74.5, 72.9), turned to -90 degrees
- moved R12 29.5 mm to (89.0, 72.0), turned to 90 degrees
- moved R47 28.9 mm to (89.0, 69.0), turned to -90 degrees
- moved U6 27.8 mm to (77.9, 55.0), turned to -90 degrees
- moved R10 19.8 mm to (89.2, 78.2), turned to 90 degrees
- moved R48 18.0 mm to (100.1, 69.1), turned to -90 degrees
- moved R56 17.4 mm to (79.0, 78.0)
- moved R11 16.7 mm to (89.2, 75.1), turned to -90 degrees
- moved R17 16.5 mm to (101.6, 72.3)
- moved U7 14.1 mm to (94.5, 73.7), turned to 180 degrees
- moved R55 11.5 mm to (75.6, 78.0)
- moved R62 10.9 mm to (66.5, 71.0), turned to 0 degrees
- moved R64 10.8 mm to (85.9, 70.7), turned to 180 degrees
- moved Q3 10.6 mm to (66.0, 77.7)
- moved R58 10.4 mm to (66.0, 74.9)
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Connections:
- J10 pad 1: Net-(J10-Pad1) -> Net-(U12-Pad3)
- J7 pad 1: Net-(J7-Pad1) -> Net-(U9-Pad3)
- J8 pad 1: Net-(J8-Pad1) -> Net-(U10-Pad3)
- J8 pad 2: Net-(J8-Pad2) -> Net-(U10-Pad5)
- J8 pad 3: Net-(J8-Pad3) -> Net-(U10-Pad10)
- J8 pad 4: Net-(J8-Pad4) -> Net-(U10-Pad8)
- J9 pad 1: Net-(J9-Pad1) -> Net-(U11-Pad3)
- J9 pad 2: Net-(J9-Pad2) -> Net-(U11-Pad5)
- J9 pad 3: Net-(J9-Pad3) -> Net-(U11-Pad10)
- J9 pad 4: Net-(J9-Pad4) -> Net-(U11-Pad8)
- U10 pad 10: Net-(J8-Pad2) -> Net-(U10-Pad10)
- U10 pad 3: Net-(J8-Pad4) -> Net-(U10-Pad3)
- U10 pad 5: Net-(J8-Pad3) -> Net-(U10-Pad5)
- U10 pad 8: Net-(J8-Pad1) -> Net-(U10-Pad8)
- U11 pad 10: Net-(J9-Pad2) -> Net-(U11-Pad10)
- U11 pad 3: Net-(J9-Pad4) -> Net-(U11-Pad3)
- U11 pad 5: Net-(J9-Pad3) -> Net-(U11-Pad5)
- U11 pad 8: Net-(J9-Pad1) -> Net-(U11-Pad8)
- U12 pad 10: Net-(J10-Pad2) -> Net-(J10-Pad3)
- U12 pad 3: Net-(J10-Pad4) -> Net-(U12-Pad3)
- U12 pad 5: Net-(J10-Pad3) -> Net-(J10-Pad2)
- U12 pad 8: Net-(J10-Pad1) -> Net-(J10-Pad4)
- U2 pad 9: +3.3V -> /VREF
- U6 pad 1: +5V -> /VREF
- U6 pad 2: Net-(R15-Pad1) -> Net-(R66-Pad1)
- U7 pad 1: +5V -> +3.3V
- U7 pad 2: Net-(R16-Pad1) -> Net-(R15-Pad1)
- U7 pad 3: GND -> +3.3V
- U7 pad 4: /LIMIT_2 -> Net-(R16-Pad1)
- U8 pad 1: +5V -> Net-(R52-Pad2)
- U8 pad 2: Net-(R17-Pad1) -> GND
- U8 pad 3: GND -> Net-(R51-Pad2)
- U8 pad 4: /LIMIT_3 -> GND
- U9 pad 10: Net-(J7-Pad2) -> Net-(J7-Pad3)
- U9 pad 3: Net-(J7-Pad4) -> Net-(U9-Pad3)
- U9 pad 5: Net-(J7-Pad3) -> Net-(J7-Pad2)
- U9 pad 8: Net-(J7-Pad1) -> Net-(J7-Pad4)
- Y1 pad 2: /XTAL1 -> GND
Routing:
- net +3.3V: track 371.2 -> 325.9 mm, vias 4 -> 6
- net +5V: track 234.8 -> 194.1 mm, vias 3 -> 1
- net /STEP_ENA: track 170.3 -> 137.5 mm, vias 9 -> 5
- net +12V: track 162.8 -> 191.9 mm
- net /LIMIT_4: track 48.1 -> 22.6 mm
- net /LIMIT_3: track 46.3 -> 29.2 mm
- net /STEP_3: track 39.8 -> 52.6 mm
- net Net-(J4-Pad1): track 23.3 -> 11.2 mm
- net Net-(U11-Pad10): track 0.00 -> 12.1 mm, vias 0 -> 2
- net Net-(U10-Pad10): track 0.00 -> 12.1 mm, vias 0 -> 2
- net /VREF: track 0.00 -> 11.9 mm
- net Net-(J9-Pad4): track 10.2 -> 0.00 mm, vias 2 -> 0
- net /LIMIT_1: track 34.2 -> 44.2 mm
- net Net-(J8-Pad4): track 9.95 -> 0.00 mm, vias 2 -> 0
- net Net-(J14-Pad2): track 5.32 -> 15.3 mm
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
Commit message: HW fixes
Parts:
- added R68: 20K, Resistor_SMD:R_0603_1608Metric, F.Cu at (72.7, 38.6)
- added R69: 20K, Resistor_SMD:R_0603_1608Metric, F.Cu at (84.7, 32.5)
- added R70: 20K, Resistor_SMD:R_0603_1608Metric, F.Cu at (96.1, 32.5)
- added R71: 20K, Resistor_SMD:R_0603_1608Metric, F.Cu at (107.8, 32.3)
- added R72: 20K, Resistor_SMD:R_0603_1608Metric, F.Cu at (73.2, 32.5)
- C2: footprint Capacitor_SMD:CP_Elec_6.3x5.9 -> Capacitor_Tantalum_SMD:CP_EIA-7343-31_Kemet-D
- D4, L1, R46, RV5, U1: moved to F.Cu
- moved R31 35.4 mm to (107.2, 46.6), turned to -90 degrees
- moved C2 28.5 mm to (124.2, 72.3), turned to -90 degrees
- moved D4 21.0 mm to (120.8, 81.0), turned to -90 degrees
- moved FID4 17.1 mm to (127.6, 67.3)
- moved RV5 8.56 mm to (105.0, 74.3), turned to 90 degrees
- moved L1 5.73 mm to (104.9, 68.1)
- moved R17 3.54 mm to (100.1, 69.1)
- moved R46 3.00 mm to (107.6, 73.2)
- moved R48 2.82 mm to (98.0, 67.2), turned to 0 degrees
- moved C20 1.54 mm to (111.5, 32.3), turned to 180 degrees
- moved C16 1.17 mm to (87.6, 32.0)
- moved C14 1.02 mm to (76.0, 32.0)
- moved C18 1.00 mm to (99.1, 31.9)
- moved U1 0.96 mm to (116.8, 70.2)
- moved C13 0.30 mm to (105.7, 42.4)
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Connections:
- JP5 pad 2: Net-(JP5-Pad2) -> Net-(U10-Pad15)
- R31 pad 1: +3.3V -> /STEP_ENA
- R31 pad 2: /STEP_ENA -> +3.3V
- R33 pad 1: +3.3V -> GND
- R33 pad 2: /STEP_ENA -> Net-(U10-Pad15)
- R35 pad 1: +3.3V -> GND
- R35 pad 2: /STEP_ENA -> Net-(JP7-Pad2)
- R37 pad 1: +3.3V -> GND
- R37 pad 2: /STEP_ENA -> Net-(JP9-Pad2)
- U10 pad 15: Net-(JP5-Pad2) -> Net-(U10-Pad15)
Routing:
- net Net-(D4-Pad1): track 13.1 -> 25.6 mm
- net +5V: track 194.1 -> 183.6 mm, vias 1 -> 4
- net Net-(R46-Pad1): track 18.5 -> 10.3 mm
- net /LIGHT_POWER: track 40.1 -> 34.5 mm
- net Net-(J12-Pad1): track 23.4 -> 28.6 mm
- net Net-(J5-Pad1): track 14.8 -> 19.2 mm
- net Net-(U10-Pad15): track 0.00 -> 4.28 mm
- net GND: track 57.3 -> 53.1 mm, vias 48 -> 46
- net +12V: track 191.9 -> 187.9 mm, vias 2 -> 6
- net +3.3V: track 325.9 -> 328.6 mm
- net Net-(JP5-Pad2): track 2.12 -> 0.00 mm
- net Net-(U9-Pad15): track 2.27 -> 4.38 mm
- net Net-(JP7-Pad2): track 2.07 -> 4.08 mm
- net Net-(U12-Pad16): track 1.85 -> 3.84 mm
- net Net-(JP9-Pad2): track 1.92 -> 3.91 mm
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
Commit message: Some tweaks
Parts:
- added Q6: AO3401A, Package_TO_SOT_SMD:SOT-23, B.Cu at (116.0, 40.0)
- added R73: 100, Resistor_SMD:R_0603_1608Metric, B.Cu at (115.5, 42.7)
- added R74: 47K, Resistor_SMD:R_0603_1608Metric, B.Cu at (112.9, 39.8)
- R31: value 20K -> 10K
Connections:
- A1 pad 9: /STEP_ENA -> /Stepper Drivers/POLOLU_ENA
- A2 pad 9: /STEP_ENA -> /Stepper Drivers/POLOLU_ENA
Routing:
- net /Stepper Drivers/POLOLU_ENA: track 0.00 -> 26.5 mm
- net /STEP_ENA: track 138.3 -> 118.2 mm
- net +3.3V: track 328.6 -> 333.4 mm, vias 6 -> 7
- net Net-(Q6-Pad2): track 0.00 -> 1.99 mm

Commit message: PCB v0.3 went to production
Parts:
- added D10: TCST-1103, TCST:TCST-1103, B.Cu at (90.8, 95.7)
- added D11: TCST-1103, TCST:TCST-1103, B.Cu at (104.3, 95.6)
- added D12: TCST-1103, TCST:TCST-1103, B.Cu at (131.3, 95.5)
- added D9: TCST-1103, TCST:TCST-1103, B.Cu at (64.2, 95.8)
- added J20: Endstop_Sensor_L, Connector_JST:JST_GH_SM03B-GHS-TB_1x03-1MP_P1.25mm_Horizontal, F.Cu at (72.8, 95.7)
- added J21: Endstop_Sensor_R, Connector_JST:JST_GH_SM03B-GHS-TB_1x03-1MP_P1.25mm_Horizontal, F.Cu at (82.3, 95.6)
- added J22: Endstop_Sensor_R, Connector_JST:JST_GH_SM03B-GHS-TB_1x03-1MP_P1.25mm_Horizontal, F.Cu at (113.0, 95.5)
- added J23: Endstop_Sensor_L, Connector_JST:JST_GH_SM03B-GHS-TB_1x03-1MP_P1.25mm_Horizontal, F.Cu at (122.7, 95.5)
- added R75: 200, Resistor_SMD:R_0603_1608Metric, F.Cu at (65.4, 95.6)
- added R76: 200, Resistor_SMD:R_0603_1608Metric, F.Cu at (89.9, 95.8)
- added R77: 200, Resistor_SMD:R_0603_1608Metric, F.Cu at (130.4, 95.7)
- added R78: 200, Resistor_SMD:R_0603_1608Metric, F.Cu at (105.5, 95.5)
- J12, J3, J4, J5: footprint Connector_JST:JST_EH_B2B-EH-A_1x02_P2.50mm_Vertical -> Connector_JST:JST_GH_BM03B-GHS-TBT_1x03-1MP_P1.25mm_Vertical
- J6: footprint Connector_JST:JST_EH_B2B-EH-A_1x02_P2.50mm_Vertical -> Connector_JST:JST_GH_BM02B-GHS-TBT_1x02-1MP_P1.25mm_Vertical
- moved R9 2.95 mm to (128.4, 65.2), turned to 180 degrees
- moved J6 2.25 mm to (128.6, 82.4), turned to 180 degrees
- moved D4 2.18 mm to (122.9, 81.0)
- moved J12 2.12 mm to (117.7, 81.6)
- moved J3 1.94 mm to (100.6, 81.6)
- moved J5 1.69 mm to (112.0, 81.6)
- moved J4 1.59 mm to (106.3, 81.6)
- moved J16 1.52 mm to (91.9, 82.7)
- moved J15 1.32 mm to (83.5, 82.7)
- moved J14 1.07 mm to (75.2, 82.8)
- moved Q1 0.93 mm to (128.7, 73.8)
- moved J13 0.89 mm to (66.8, 82.7)
- moved U5 0.84 mm to (132.9, 67.1)
- moved JP1 0.74 mm to (135.4, 51.4)
- moved JP10 0.74 mm to (131.5, 56.4)
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Connections:
- R65 pad 1: +3.3V -> +5V
Routing:
- net +5V: track 183.6 -> 233.4 mm, vias 4 -> 6
- net +3.3V: track 333.4 -> 351.2 mm, vias 7 -> 5
- net Net-(D9-Pad3): track 0.00 -> 14.9 mm
- net Net-(D10-Pad3): track 0.00 -> 12.8 mm
- net Net-(J21-Pad3): track 0.00 -> 11.4 mm
- net Net-(J23-Pad3): track 0.00 -> 9.62 mm
- net Net-(J20-Pad3): track 0.00 -> 8.29 mm
- net Net-(D11-Pad3): track 0.00 -> 8.21 mm
- net Net-(J22-Pad3): track 0.00 -> 7.39 mm
- net Net-(D11-Pad1): track 0.00 -> 4.65 mm
- net Net-(D12-Pad1): track 0.00 -> 4.33 mm
- net Net-(D12-Pad3): track 0.00 -> 3.86 mm
- net /LIGHT_POWER: track 34.5 -> 30.8 mm
- net Net-(R9-Pad2): track 2.60 -> 6.14 mm
- net Net-(D10-Pad1): track 0.00 -> 2.40 mm
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- added copper zone on B.Cu, net Net-(D10-Pad2)
- added copper zone on F.Cu, net Net-(D10-Pad2)
- added copper zone on B.Cu, net Net-(D11-Pad2)
- added copper zone on F.Cu, net Net-(D11-Pad2)
- added copper zone on B.Cu, net Net-(D12-Pad2)
- added copper zone on F.Cu, net Net-(D12-Pad2)
- added copper zone on B.Cu, net Net-(D9-Pad2)
- added copper zone on F.Cu, net Net-(D9-Pad2)
Other:
- board size 80 x 60 mm -> 80.1 x 77.3 mm
- board text added: "PNP Head v0.3 March 2023"
- board text removed: "PNP head v0.2 December 2022"
