File: hardware/stm32-head/stm32-head.kicad_sch (KiCad schematic)
At the start: 99 parts, among them J1 POWER, J11 SWD, J12 LIMIT_4, J13 SOLENOID1, J14 SOLENOID2, J15 SOLENOID3, J16 SOLENOID4, J19 LED, J2 RS-485, J3 LIMIT_1, J4 LIMIT_2, J5 LIMIT_3, J6 LIGHT, Q1 IRF540N, Q2 AO3400A, Q3 AO3400A, Q4 AO3400A, Q5 AO3400A, SW1 RESET, U1 LM2596S-ADJ, U13 PC817, U14 PC817, U15 PC817, U16 PC817, U17 PC817, U2 STM32F103C8Tx, U3 AMS1117-3.3, U4 MAX483E, U5 PC817, U6 PC817, U7 PC817, U8 PC817, Y1 8Mhz

Commit message: Board fixes
Parts:
- removed U13, U14, U15, U16, U17, U6, U7, U8: PC817, Package_DIP:SMDIP-4_W9.53mm, symbol Isolator:PC817
- removed Y1: 8Mhz, Crystal:Crystal_SMD_5032-2Pin_5.0x3.2mm, symbol Device:Crystal
- added FID1, FID2, FID3, FID4: Fiducial, Fiducial:Fiducial_0.5mm_Mask1mm, symbol Mechanical:Fiducial
- added R65: 1K, Resistor_SMD:R_0603_1608Metric, symbol Device:R
- added R66: 10K, Resistor_SMD:R_0603_1608Metric, symbol Device:R
- added R67: 32K, Resistor_SMD:R_0603_1608Metric, symbol Device:R
- added U6: TL431DBZ, Package_TO_SOT_SMD:SOT-23, symbol Reference_Voltage:TL431DBZ
- added U7, U8: TLP291-4, Package_SO:SOIC-16_4.55x10.3mm_P1.27mm, symbol Isolator:TLP291-4
- added Y1: 8Mhz, Crystal:Crystal_SMD_3225-4Pin_3.2x2.5mm, symbol Device:Crystal_GND24
- Q1: footprint Package_TO_SOT_THT:TO-220-3_Vertical -> Package_TO_SOT_SMD:TO-252-3_TabPin2
- R2, R61, R62, R63, R64: value 100 -> 510
- R49, R50, R51, R52, R9: value 100 -> 150
Connections:
- net +3.3V: now also R65.1, U7.1, U7.3, U7.5, U7.7, U8.10, U8.12, U8.14, U8.16; no longer U2.9 (VDDA)
- net GND: now also R67.2, U6.3 (A), U7.11, U7.13, U7.15, U7.9, U8.2, U8.4, U8.6, U8.8, Y1.2, Y1.4
- net LIMIT_1: now also U7.16
- net LIMIT_2: now also U7.14
- net LIMIT_3: now also U7.12
- net LIMIT_4: now also U7.10
- net XTAL1: now also Y1.3
- net XTAL2: now also Y1.1
- net at R53.1: now also U8.9
- net at R55.1: now also U8.13
- net at R48.1: now also U7.8
- net at R52.2: now also U8.1
- net at R56.1: now also U8.15
- net at R51.2: now also U8.3
- net at R54.1: now also U8.11
- net at R50.2: now also U8.5
- net at R17.1: now also U7.6
- net at R16.1: now also U7.4
- net at R15.1: now also U7.2
- net at R49.2: now also U8.7
- new net: R66.1, R67.1, U6.2 (REF)
- new net VREF: R65.2, R66.2, U2.9 (VDDA), U6.1 (K)
Other:
- moved on the sheet: C6, C7, C8, C9, H1, H2, H3, H4, J11

Commit message: HW fixes
Parts:
- C2: footprint Capacitor_SMD:CP_Elec_6.3x5.9 -> Capacitor_Tantalum_SMD:CP_EIA-7343-31_Kemet-D
Changed lines of the file:
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@@
   (symbol (lib_id "Device:R") (at 27.686 122.936 90) (unit 1)
     (in_bom yes) (on_board yes)
-    (property "Reference" "R65" (id 0) (at 23.876 121.412 90))
+    (property "Reference" "R65" (id 0) (at 27.686 120.65 90))
     (property "Value" "1K" (id 1) (at 27.686 122.936 90))
     (property "Footprint" "Resistor_SMD:R_0603_1608Metric" (id 2) (at 27.686 124.714 90)
@@
   (symbol (lib_id "Device:R") (at 28.194 133.604 0) (unit 1)
     (in_bom yes) (on_board yes)
-    (property "Reference" "R67" (id 0) (at 23.622 131.318 0)
+    (property "Reference" "R67" (id 0) (at 30.48 135.636 90)
       (effects (font (size 1.27 1.27)) (justify left))
     )
@@
       (effects (font (size 1.27 1.27)) (justify left))
     )
-    (property "Footprint" "Capacitor_SMD:CP_Elec_6.3x5.9" (id 2) (at 59.1312 194.31 0)
+    (property "Footprint" "Capacitor_Tantalum_SMD:CP_EIA-7343-31_Kemet-D" (id 2) (at 59.1312 194.31 0)
       (effects (font (size 1.27 1.27)) hide)
     )
@@
   (symbol (lib_id "Device:R") (at 27.686 125.984 90) (unit 1)
     (in_bom yes) (on_board yes)
-    (property "Reference" "R66" (id 0) (at 23.622 124.968 90))
+    (property "Reference" "R66" (id 0) (at 21.59 126.238 90))
     (property "Value" "10K" (id 1) (at 27.686 125.984 90))
     (property "Footprint" "Resistor_SMD:R_0603_1608Metric" (id 2) (at 27.686 127.762 90)
@@
       (reference "#PWR020") (unit 1) (value "GND") (footprint "")
     )
+    (path "/92493782-b039-48c6-8181-4f20920a88e0/bc55ba4e-df78-4524-9f40-93c1314218ed"
+      (reference "#PWR021") (unit 1) (value "GND") (footprint "")
+    )
     (path "/a5bf0c14-2a69-40b9-bf55-1e74cccf3e26"
       (reference "#PWR022") (unit 1) (value "+3.3V") (footprint "")
@@
       (reference "#PWR026") (unit 1) (value "GND") (footprint "")
     )
+    (path "/92493782-b039-48c6-8181-4f20920a88e0/7f619eaa-36ef-4da1-8f57-7224c9db96d8"
+      (reference "#PWR027") (unit 1) (value "GND") (footprint "")
+    )
     (path "/5c4a6d77-bee0-411c-9f15-86390968863b"
       (reference "#PWR028") (unit 1) (value "GND") (footprint "")
@@
       (reference "#PWR052") (unit 1) (value "GND") (footprint "")
     )
+    (path "/92493782-b039-48c6-8181-4f20920a88e0/baf5bbd5-1f16-4d3a-ac32-88a0b3e785a5"
+      (reference "#PWR053") (unit 1) (value "GND") (footprint "")
+    )
+    (path "/92493782-b039-48c6-8181-4f20920a88e0/cf92db11-0afb-4569-8022-14844ff29301"
+      (reference "#PWR054") (unit 1) (value "+3.3V") (footprint "")
+    )
+    (path "/92493782-b039-48c6-8181-4f20920a88e0/d0be26e9-583c-4fa6-a29b-dd044af74438"
+      (reference "#PWR055") (unit 1) (value "GND") (footprint "")
+    )
+    (path "/92493782-b039-48c6-8181-4f20920a88e0/694cfe6d-6c1f-49c6-a46b-a760728ee874"
+      (reference "#PWR056") (unit 1) (value "+3.3V") (footprint "")
+    )
+    (path "/92493782-b039-48c6-8181-4f20920a88e0/b51fcce7-43dd-429a-adbc-61d13964bb2d"
+      (reference "#PWR057") (unit 1) (value "+3.3V") (footprint "")
+    )
+    (path "/92493782-b039-48c6-8181-4f20920a88e0/59daa1aa-b113-4760-a686-ac42357b8f33"
+      (reference "#PWR058") (unit 1) (value "+3.3V") (footprint "")
+    )
     (path "/36243262-c60c-4823-b134-a9f302f927ff"
       (reference "#PWR0101") (unit 1) (value "GND") (footprint "")
@@
       (reference "#PWR0137") (unit 1) (value "+12V") (footprint "")
     )
+    (path "/92493782-b039-48c6-8181-4f20920a88e0/8614f33a-7912-411f-8d34-0d413d4917e9"
+      (reference "#PWR0138") (unit 1) (value "+3.3V") (footprint "")
+    )
+    (path "/92493782-b039-48c6-8181-4f20920a88e0/0784c8e7-5728-4586-b1e8-47462d42c978"
+      (reference "#PWR?") (unit 1) (value "GND") (footprint "")
+    )
     (path "/92493782-b039-48c6-8181-4f20920a88e0/6b9d3db7-eeaa-432e-86b6-c2d683baaf45"
       (reference "A1") (unit 1) (value "DRV8825") (footprint "Module:Pololu_Breakout-16_15.2x20.3mm")
@@
     )
     (path "/7e1d0587-cd17-4aca-aa52-4cdb36cae601"
-      (reference "C2") (unit 1) (value "220uF") (footprint "Capacitor_SMD:CP_Elec_6.3x5.9")
+      (reference "C2") (unit 1) (value "220uF") (footprint "Capacitor_Tantalum_SMD:CP_EIA-7343-31_Kemet-D")
     )
     (path "/f27eebcc-9e24-455a-b6df-2a17cb319e5a"
@@
       (reference "Q5") (unit 1) (value "AO3400A") (footprint "Package_TO_SOT_SMD:SOT-23")
     )
+    (path "/92493782-b039-48c6-8181-4f20920a88e0/76d4d68d-1cc6-4380-93a3-08bf06c7b857"
+      (reference "Q?") (unit 1) (value "AO3400A") (footprint "Package_TO_SOT_SMD:SOT-23")
+    )
     (path "/30f4f394-b9dc-4e13-a469-325f78b86a5c"
       (reference "R1") (unit 1) (value "1K") (footprint "Resistor_SMD:R_0603_1608Metric")
@@
       (reference "R32") (unit 1) (value "47K") (footprint "Resistor_SMD:R_0603_1608Metric")
     )
-    (path "/92493782-b039-48c6-8181-4f20920a88e0/f84f46ff-f103-48d9-9b49-baa8750c4558"
+    (path "/92493782-b039-48c6-8181-4f20920a88e0/380d08b3-16d8-40b5-905f-2e6ed7333e7e"
       (reference "R33") (unit 1) (value "20K") (footprint "Resistor_SMD:R_0603_1608Metric")
     )
@@
       (reference "R34") (unit 1) (value "47K") (footprint "Resistor_SMD:R_0603_1608Metric")
     )
-    (path "/92493782-b039-48c6-8181-4f20920a88e0/a68b83bd-0cbf-41b7-88c4-c9fb47418a8a"
+    (path "/92493782-b039-48c6-8181-4f20920a88e0/b603762f-ec05-4e1c-819d-542dd8161449"
       (reference "R35") (unit 1) (value "20K") (footprint "Resistor_SMD:R_0603_1608Metric")
     )
@@
       (reference "R36") (unit 1) (value "47K") (footprint "Resistor_SMD:R_0603_1608Metric")
     )
-    (path "/92493782-b039-48c6-8181-4f20920a88e0/888ec800-fd69-4a4d-8ef6-f8cf92b857ae"
+    (path "/92493782-b039-48c6-8181-4f20920a88e0/52384b90-987b-4c2f-87cd-2305bca33a3e"
       (reference "R37") (unit 1) (value "20K") (footprint "Resistor_SMD:R_0603_1608Metric")
     )
@@
       (reference "R67") (unit 1) (value "32K") (footprint "Resistor_SMD:R_0603_1608Metric")
     )
+    (path "/92493782-b039-48c6-8181-4f20920a88e0/67010ecc-db48-46a2-aab6-4ee4ceaab4ae"
+      (reference "R68") (unit 1) (value "20K") (footprint "Resistor_SMD:R_0603_1608Metric")
+    )
+    (path "/92493782-b039-48c6-8181-4f20920a88e0/9b07427b-3eca-40b1-9fb3-9652cd086c71"
+      (reference "R69") (unit 1) (value "20K") (footprint "Resistor_SMD:R_0603_1608Metric")
+    )
+    (path "/92493782-b039-48c6-8181-4f20920a88e0/b82796e8-d9fd-4303-969a-42d4c67d98cd"
+      (reference "R70") (unit 1) (value "20K") (footprint "Resistor_SMD:R_0603_1608Metric")
+    )
+    (path "/92493782-b039-48c6-8181-4f20920a88e0/b154f942-6f45-489a-8139-effb64b66f4f"
+      (reference "R71") (unit 1) (value "20K") (footprint "Resistor_SMD:R_0603_1608Metric")
+    )
+    (path "/92493782-b039-48c6-8181-4f20920a88e0/566645cb-6304-4955-b8ef-fa0255e9c060"
+      (reference "R72") (unit 1) (value "20K") (footprint "Resistor_SMD:R_0603_1608Metric")
+    )
+    (path "/92493782-b039-48c6-8181-4f20920a88e0/3e15d7e0-f02f-4d6c-b17b-0e4dc3635df7"
+      (reference "R?") (unit 1) (value "5K") (footprint "Resistor_SMD:R_0603_1608Metric")
+    )
+    (path "/92493782-b039-48c6-8181-4f20920a88e0/9186f09f-c04a-4499-a97d-a9b36baef4da"
+      (reference "R?") (unit 1) (value "100") (footprint "Resistor_SMD:R_0603_1608Metric")
+    )
     (path "/92493782-b039-48c6-8181-4f20920a88e0/7133a6f3-e0ec-424f-8733-ec6f74d56e45"

Commit message: PCB v0.3 went to production
Parts:
- removed J12: LIMIT_4, Connector_JST:JST_EH_B2B-EH-A_1x02_P2.50mm_Vertical, symbol Connector:Conn_01x02_Female
- removed J3: LIMIT_1, Connector_JST:JST_EH_B2B-EH-A_1x02_P2.50mm_Vertical, symbol Connector:Conn_01x02_Female
- removed J4: LIMIT_2, Connector_JST:JST_EH_B2B-EH-A_1x02_P2.50mm_Vertical, symbol Connector:Conn_01x02_Female
- removed J5: LIMIT_3, Connector_JST:JST_EH_B2B-EH-A_1x02_P2.50mm_Vertical, symbol Connector:Conn_01x02_Female
- added D10, D11, D12, D9: TCST-1103, TCST:TCST-1103, symbol TCST:TCST-1103
- added J12: LIMIT_4, Connector_JST:JST_GH_BM03B-GHS-TBT_1x03-1MP_P1.25mm_Vertical, symbol Connector:Conn_01x03_Female
- added J20, J23: Endstop_Sensor_L, Connector_JST:JST_GH_SM03B-GHS-TB_1x03-1MP_P1.25mm_Horizontal, symbol Connector:Conn_01x03_Female
- added J21, J22: Endstop_Sensor_R, Connector_JST:JST_GH_SM03B-GHS-TB_1x03-1MP_P1.25mm_Horizontal, symbol Connector:Conn_01x03_Female
- added J3: LIMIT_1, Connector_JST:JST_GH_BM03B-GHS-TBT_1x03-1MP_P1.25mm_Vertical, symbol Connector:Conn_01x03_Female
- added J4: LIMIT_2, Connector_JST:JST_GH_BM03B-GHS-TBT_1x03-1MP_P1.25mm_Vertical, symbol Connector:Conn_01x03_Female
- added J5: LIMIT_3, Connector_JST:JST_GH_BM03B-GHS-TBT_1x03-1MP_P1.25mm_Vertical, symbol Connector:Conn_01x03_Female
- added R75, R76, R77, R78: 200, Resistor_SMD:R_0603_1608Metric, symbol Device:R
- J6: footprint Connector_JST:JST_EH_B2B-EH-A_1x02_P2.50mm_Vertical -> Connector_JST:JST_GH_BM02B-GHS-TBT_1x02-1MP_P1.25mm_Vertical
Connections:
- net +3.3V: now also J12.3 (Pin_3), J3.3 (Pin_3), J4.3 (Pin_3), J5.3 (Pin_3); no longer R65.1
- net +5V: now also R65.1
- net GND: now also J12.2 (Pin_2), J3.2 (Pin_2), J4.2 (Pin_2), J5.2 (Pin_2)
- net at R48.2: now also J12.1 (Pin_1)
- net at R16.2: now also J4.1 (Pin_1)
- net at R15.2: now also J3.1 (Pin_1)
- net at R17.2: now also J5.1 (Pin_1)
- new net: J20.3 (Pin_3), R75.1
- new net: D9.1 (E+), R75.2
- new net: D12.3 (DC), J23.1 (Pin_1)
- new net: D12.2 (E-), D12.4 (DE), J23.2 (Pin_2)
- new net: J23.3 (Pin_3), R77.1
- new net: J21.3 (Pin_3), R76.1
- new net: D10.1 (E+), R76.2
- new net: D11.3 (DC), J22.1 (Pin_1)
- new net: D11.2 (E-), D11.4 (DE), J22.2 (Pin_2)
- new net: J22.3 (Pin_3), R78.1
- new net: D9.2 (E-), D9.4 (DE), J20.2 (Pin_2)
- new net: D9.3 (DC), J20.1 (Pin_1)
- new net: D10.3 (DC), J21.1 (Pin_1)
- new net: D10.2 (E-), D10.4 (DE), J21.2 (Pin_2)
- new net: D12.1 (E+), R77.2
- new net: D11.1 (E+), R78.2
Other:
- moved on the sheet: R15, R16, R17, R48
